File: pcb/Schematic.kicad_sch (KiCad schematic)
At the start: 42 parts, among them J1 Motor, J2 Load cell, J3 Optic_spin_ctl 1OUT 2GND 3IN, J4 tank_presence_led_emitter, J5 tank_pres_led_recv, J6 SWD VCC, CLK, IO, GND, Q6 NPN, Q8 NPN, U1 6210A, U2 1117A

Commit message: Added n32g43x bsp, added first test button-blinking firmware
Parts:
- added BZ1: Buzzer, Package_DFN_QFN:Texas_RGP0020D_VQFN-20-1EP_4x4mm_P0.5mm_EP2.7x2.7mm_ThermalVias, symbol Device:Buzzer
- added J7: button_connector, Display:HY1602E, symbol Connector:Conn_01x06_Pin
- added Q10, Q11, Q12, Q7: NPN, Package_DFN_QFN:Nordic_AQFN-94-1EP_7x7mm_P0.4mm, symbol Simulation_SPICE:NPN
Connections:
- net GND: now also J7.6 (Pin_6), Q10.3 (E), Q11.3 (E), Q12.3 (E), Q7.3 (E)
- net VCC 5V: now also BZ1.1 (+), J7.1 (Pin_1)
- net BUZZER: now reaches N32G1.17 (PA7)
- net BUZZER: now also Q7.2 (B)
- net BTN_LED_R: now reaches N32G1.21 (PB10)
- net BTN_LED_R: now also Q10.2 (B)
- net BTN_LED_G: now reaches N32G1.22 (PB11)
- net BTN_LED_G: now also Q12.2 (B)
- net BTN_LED_B: now reaches N32G1.25 (PB12)
- net BTN_LED_B: now also Q11.2 (B)
- net BTN_KEY: now reaches N32G1.26 (PB13)
- net BTN_KEY: now also J7.5 (Pin_5)
- new net: J7.2 (Pin_2), Q10.1 (C)
- new net: J7.3 (Pin_3), Q12.1 (C)
- new net: J7.4 (Pin_4), Q11.1 (C)
- new net: BZ1.2 (-), Q7.1 (C)
